File: pcb/flight_computer/mcu.kicad_sch (KiCad schematic)
At the start: 26 parts, among them J3 SWD (ARM 10-pin 1.27mm), J4 USB-C, SW1 reset, U2 STM32F405RGT6, U3 USBLC6-2SC6, Y1 8MHz

Commit message: Flight computer: pack-voltage sense, BOM re-verified, pre-fab audit
- PA0 reads the 2S pack through R34/R35 (100k/33k) + C33; nothing could before.
- 32 of 39 BOM lines confirmed on LCSC product pages; SW1 -> TL3342F160QG
  (C2886898) since the reel part is out of stock.
- R8 pinned in layout.py MANUAL_FIXUP after relax() threw it 20.8 mm.
- pcb/README.md 'What is not done' rewritten as the pre-order / bring-up list,
  including the mated-servo-plug height vs the 12 mm packing envelope.
Parts:
- added C33: 100nF, Capacitor_SMD:C_0402_1005Metric, symbol Device:C
- added R34: 100k, Resistor_SMD:R_0402_1005Metric, symbol Device:R
- added R35: 33k, Resistor_SMD:R_0402_1005Metric, symbol Device:R
Connections:
- net GND: now also C33.2, R35.2
- net VBAT_SENSE: now reaches U2.14 (PA0)
- net VBAT_SENSE: now also C33.1, R34.2, R35.1
- new net VBATT: R34.1
- no-connect marks 21 -> 20
